File: kicad/carte-alim.sch (KiCad schematic (older format))
At the start: 52 parts, among them P1 BATT, P10 5V, P11 5V, P12 5V, P13 5V, P14 5V, P15 5V, P16 5V, P17 3.3V, P18 3.3V, P19 3.3V, P2 BATT, P20 3.3V, P21 3.3V, P22 3.3V, P23 3.3V, P24 3.3V, P25 3.3V, P26 3.3V, P27 MASSE, P28 MASSE, P29 PILES, P3 BATT, P30 CONN_1, P31 CONN_1, P32 CONN_1, P4 BATT, P5 BATT, P6 BATT, P7 5V, P8 5V, P9 5V, U1 LM 1117 3.3, U2 OKI 78SR 5

Commit message: Validation et nettoyage du schéma
Parts:
- C1, C2, C3, C4: symbol C -> C-RESCUE-carte-alim
- D5, D6, D7: symbol LED -> LED-RESCUE-carte-alim
- R1, R2, R3: symbol R -> R-RESCUE-carte-alim

Commit message: Association composants
Parts:
- C1, C2, C3, C4: footprint (none) -> Capacitors_THT:C_Rect_L7.0mm_W3.5mm_P2.50mm_P5.00mm
- C5, C6, C7, C8: footprint (none) -> Capacitors_THT:CP_Radial_D10.0mm_P2.50mm_P5.00mm
- D1, D2, D3, D4: footprint (none) -> Diodes_THT:D_A-405_P7.62mm_Horizontal
- D5, D6, D7: footprint (none) -> LEDs:LED_D3.0mm
- P1, P10, P11, P12, P13, P14, P15, P16, P17, P18, P19, P2, P20, P21, P22, P23, P24, P25, P26, P29, P3, P4, P5, P6, P7, P8, P9: footprint (none) -> EPSA_Connect:KK_2C
- P27, P28: footprint (none) -> Pin_Headers:Pin_Header_Straight_1x08_Pitch2.54mm
- P30, P31, P32: footprint (none) -> Mounting_Holes:MountingHole_3.2mm_M3_Pad
- R1, R2, R3: footprint (none) -> Resistors_THT:R_Axial_DIN0207_L6.3mm_D2.5mm_P7.62mm_Horizontal
- U1, U2: footprint (none) -> TO_SOT_Packages_THT:TO-220-3_Vertical

Commit message: Utilisation de diodes avec un pas de 10mm au lieu de 7,5mm
Parts:
- D1, D2, D3, D4: footprint Diodes_THT:D_A-405_P7.62mm_Horizontal -> Diodes_THT:D_DO-15_P10.16mm_Horizontal
Changed lines of the file:
@@
 F 0 "D3" H 9800 4750 40  0000 C CNN
 F 1 "5A" H 9800 4550 40  0000 C CNN
-F 2 "Diodes_THT:D_A-405_P7.62mm_Horizontal" H 9800 4650 60  0001 C CNN
+F 2 "Diodes_THT:D_DO-15_P10.16mm_Horizontal" H 9800 4650 60  0001 C CNN
 F 3 "" H 9800 4650 60  0001 C CNN
 	1    9800 4650
@@
 F 0 "D4" H 9800 5150 40  0000 C CNN
 F 1 "5A" H 9800 4950 40  0000 C CNN
-F 2 "Diodes_THT:D_A-405_P7.62mm_Horizontal" H 9800 5050 60  0001 C CNN
+F 2 "Diodes_THT:D_DO-15_P10.16mm_Horizontal" H 9800 5050 60  0001 C CNN
 F 3 "" H 9800 5050 60  0001 C CNN
 	1    9800 5050
@@
 F 0 "D2" H 8550 5150 40  0000 C CNN
 F 1 "5A" H 8550 4950 40  0000 C CNN
-F 2 "Diodes_THT:D_A-405_P7.62mm_Horizontal" H 8550 5050 60  0001 C CNN
+F 2 "Diodes_THT:D_DO-15_P10.16mm_Horizontal" H 8550 5050 60  0001 C CNN
 F 3 "" H 8550 5050 60  0001 C CNN
 	1    8550 5050
@@
 F 0 "D1" H 8550 4750 40  0000 C CNN
 F 1 "5A" H 8550 4550 40  0000 C CNN
-F 2 "Diodes_THT:D_A-405_P7.62mm_Horizontal" H 8550 4650 60  0001 C CNN
+F 2 "Diodes_THT:D_DO-15_P10.16mm_Horizontal" H 8550 4650 60  0001 C CNN
 F 3 "" H 8550 4650 60  0001 C CNN
 	1    8550 4650

Commit message: Mise en qualité du typon
Parts:
- removed D1, D2, D3, D4: 5A, Diodes_THT:D_DO-15_P10.16mm_Horizontal, symbol DIODE
- removed P1: BATT, EPSA_Connect:KK_2C, symbol CONN_2
- removed P21, P26: 3.3V, EPSA_Connect:KK_2C, symbol CONN_2
- added D1, D2, D3, D4: 5A, Diodes_THT:D_DO-15_P10.16mm_Horizontal, symbol D_ALT
- added P33: CONN_1, Mounting_Holes:MountingHole_3.2mm_M3_Pad, symbol CONN_1
Connections:
- wire segments 92 -> 90
- no-connect marks 3 -> 4

Commit message: Schématique avec connecteurs multi-tensions
Parts:
- removed C1: 100n, Capacitors_THT:C_Rect_L7.0mm_W3.5mm_P2.50mm_P5.00mm, symbol C-RESCUE-carte-alim
- removed C5: 100u, Capacitors_THT:CP_Radial_D10.0mm_P2.50mm_P5.00mm, symbol CAPAPOL
- removed D1, D2, D3, D4: 5A, Diodes_THT:D_DO-15_P10.16mm_Horizontal, symbol D_ALT
- removed D5, D6, D7: GREEN, LEDs:LED_D3.0mm, symbol LED-RESCUE-carte-alim
- removed P10, P11, P12, P13, P14, P15, P16, P7, P8, P9: 5V, EPSA_Connect:KK_2C, symbol CONN_2
- removed P17, P18, P19, P20, P22, P23, P24, P25: 3.3V, EPSA_Connect:KK_2C, symbol CONN_2
- removed P2, P3, P4, P5, P6: BATT, EPSA_Connect:KK_2C, symbol CONN_2
- removed P28: MASSE, Pin_Headers:Pin_Header_Straight_1x08_Pitch2.54mm, symbol CONN_8
- added D1: YELLOW, LEDs:LED_D3.0mm, symbol LED_ALT
- added D2: RED, LEDs:LED_D3.0mm, symbol LED_ALT
- added D3: ORANGE, LEDs:LED_D3.0mm, symbol LED_ALT
- added J1, J10, J2, J3, J4, J5, J6, J7, J8, J9: PWR_OUT, Connectors_Molex:Molex_MiniFit-JR-5569-04A2_2x02x4.20mm_Angled, symbol Conn_02x02_Odd_Even
- added P7: +5V, Pin_Headers:Pin_Header_Straight_1x08_Pitch2.54mm, symbol CONN_8
- added P8: +3.3V, Pin_Headers:Pin_Header_Straight_1x08_Pitch2.54mm, symbol CONN_8
- P1: renamed from P33; value CONN_1 -> MECA
- P2: renamed from P30; value CONN_1 -> MECA
- P3: renamed from P31; value CONN_1 -> MECA
- P4: renamed from P29; footprint EPSA_Connect:KK_2C -> Connectors_Molex:Molex_MiniFit-JR-5569-02A2_2x01x4.20mm_Angled
- P5: renamed from P32; value CONN_1 -> MECA
- U1, U2: footprint TO_SOT_Packages_THT:TO-220-3_Vertical -> TO_SOT_Packages_THT:TO-220-3_Horizontal
- renumbered C3 to C1, C7 to C2, C2 to C3, C6 to C4, C4 to C5, C8 to C6, P27 to P6, R3 to R1, R1 to R2, R2 to R3
Connections:
- wire segments 90 -> 83
Other:
- note added: "Branchement batteries"
- note added: "Bus d'alimentation"
- note added: "Convensions couleurs :\n1 - Noir : masse\n2 - Rouge - +5V\n3 - Orange : +3.3V\n4 - Jaune : BATT"
- note removed: "Branchement piles\nRedresseur pour éviter de cramer les régulateurs"
- note removed: "Bus de masse"
- note removed: "Connecteurs pour branchement vers autres cartes\n(on double pour prévoir large pour les années suivantes)"

Commit message: Réalisation du typon avec connecteurs Mini-Fit
Parts:
- U1, U2: footprint TO_SOT_Packages_THT:TO-220-3_Horizontal -> Project:TO-220-3_Horizontal_Radiat
Other:
- note added: "Convensions couleurs :\n1 - Noir : masse\n2 - Rouge : +5V\n3 - Orange : +3.3V\n4 - Jaune : BATT"
- note removed: "Convensions couleurs :\n1 - Noir : masse\n2 - Rouge - +5V\n3 - Orange : +3.3V\n4 - Jaune : BATT"
