File: kicad/carte-alim.sch (KiCad schematic (older format))
At the start: 32 parts, among them J1 PWR_OUT, J10 PWR_OUT, J2 PWR_OUT, J3 PWR_OUT, J4 PWR_OUT, J5 PWR_OUT, J6 PWR_OUT, J7 PWR_OUT, J8 PWR_OUT, J9 PWR_OUT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

Commit message: Reprise du schéma pour corriger bug d'affichage
Parts:
- removed C1, C3, C5: 100n, Capacitors_THT:C_Rect_L7.0mm_W3.5mm_P2.50mm_P5.00mm, symbol C-RESCUE-carte-alim
- removed C2, C4, C6: 100u, Capacitors_THT:CP_Radial_D10.0mm_P2.50mm_P5.00mm, symbol CAPAPOL
- removed D1: YELLOW, LEDs:LED_D3.0mm, symbol LED_ALT
- removed D2: RED, LEDs:LED_D3.0mm, symbol LED_ALT
- removed D3: ORANGE, LEDs:LED_D3.0mm, symbol LED_ALT
- removed J1, J2, J8, J9: PWR_OUT, Connectors_Molex:Molex_MiniFit-JR-5569-04A2_2x02x4.20mm_Angled, symbol Conn_02x02_Odd_Even
- removed P1, P2, P3, P5: MECA, Mounting_Holes:MountingHole_3.2mm_M3_Pad, symbol CONN_1
- removed P4: PILES, Connectors_Molex:Molex_MiniFit-JR-5569-02A2_2x01x4.20mm_Angled, symbol CONN_2
- removed P6: MASSE, Pin_Headers:Pin_Header_Straight_1x08_Pitch2.54mm, symbol CONN_8
- removed P7: +5V, Pin_Headers:Pin_Header_Straight_1x08_Pitch2.54mm, symbol CONN_8
- removed P8: +3.3V, Pin_Headers:Pin_Header_Straight_1x08_Pitch2.54mm, symbol CONN_8
- removed R1: 680, Resistors_THT:R_Axial_DIN0207_L6.3mm_D2.5mm_P7.62mm_Horizontal, symbol R-RESCUE-carte-alim
- removed R2, R3: 470, Resistors_THT:R_Axial_DIN0207_L6.3mm_D2.5mm_P7.62mm_Horizontal, symbol R-RESCUE-carte-alim
- removed U1: LM 1117 3.3, Project:TO-220-3_Horizontal_Radiat, symbol LM317T
- removed U2: OKI 78SR 5, Project:TO-220-3_Horizontal_Radiat, symbol 7805
- added C1, C3, C4: 100n, Capacitors_THT:C_Rect_L7.0mm_W3.5mm_P2.50mm_P5.00mm, symbol C
- added C2, C5, C6: 100u, Capacitors_THT:CP_Radial_D10.0mm_P2.50mm_P5.00mm, symbol CP
- added D1: YELLOW, LEDs:LED_D3.0mm, symbol LED
- added D2: RED, LEDs:LED_D3.0mm, symbol LED
- added D3: ORANGE, LEDs:LED_D3.0mm, symbol LED
- added J1, J2, J8, J9: MECA, Mounting_Holes:MountingHole_3.2mm_M3_Pad, symbol Conn_01x01
- added J10, J11, J12, J13: PWR_OUT, Connectors_Molex:Molex_MiniFit-JR-5569-04A2_2x02x4.20mm_Angled, symbol Conn_02x02_Odd_Even
- added J15: PILES, Connectors_Molex:Molex_MiniFit-JR-5569-02A2_2x01x4.20mm_Angled, symbol Conn_01x02
- added J16: GND, Pin_Headers:Pin_Header_Straight_1x08_Pitch2.54mm, symbol Conn_01x08
- added J17: +5V, Pin_Headers:Pin_Header_Straight_1x08_Pitch2.54mm, symbol Conn_01x08
- added J18: +3.3V, Pin_Headers:Pin_Header_Straight_1x08_Pitch2.54mm, symbol Conn_01x08
- added R1: 680, Resistors_THT:R_Axial_DIN0411_L9.9mm_D3.6mm_P7.62mm_Vertical, symbol R
- added R2, R3: 470, Resistors_THT:R_Axial_DIN0411_L9.9mm_D3.6mm_P7.62mm_Vertical, symbol R
- added U1: LM1117-3.3, symbol LM1117-3.3
- added U2: OKI 78SR 5, symbol L7805
- renumbered J10 to J14
Connections:
- wire segments 83 -> 76
