File: kicad/carte-alim.kicad_pcb (KiCad board)
At the start: 4 copper layers, 96.5 x 45.7 mm, 32 parts, among them J1 PWR_OUT, J10 PWR_OUT, J2 PWR_OUT, J3 PWR_OUT, J4 PWR_OUT, J5 PWR_OUT, J6 PWR_OUT, J7 PWR_OUT, J8 PWR_OUT, J9 PWR_OUT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

Commit message: Mise à jour de la version dans les cartouches et la sérigraphie
Other:
- board text added: "Carte alimentation ERACL 2018 - v1.1"
- board text removed: "Carte alimentation ERACL 2018 - v1.x"
Changed lines of the file:
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@@
   (title_block
     (title "Carte alimentation")
-    (rev v1.*)
+    (date 2018-02-11)
+    (rev v1.1)
     (company "Centrale Lyon")
     (comment 1 "ERACL 2A 2018")
@@
   (gr_arc (start 121.285 66.675) (end 116.84 66.675) (angle 90) (layer Edge.Cuts) (width 0.381))
   (gr_arc (start 208.915 66.675) (end 208.915 62.23) (angle 90) (layer Edge.Cuts) (width 0.381))
-  (gr_text "Carte alimentation ERACL 2018 - v1.x" (at 177.165 85.09) (layer F.SilkS)
+  (gr_text "Carte alimentation ERACL 2018 - v1.1" (at 177.165 85.09) (layer F.SilkS)
     (effects (font (size 2 1.5) (thickness 0.2)))
   )
